Commit message: Release Training Panel V3.0.1

File: test_7_description/test_7_description/urdf/test_7.urdf (robot description, URDF)
Before this commit: robot test_7, 25 links, 24 joints
Joints:
- removed joint Rigid 17
- removed joint Rigid 18
- removed joint Rigid 21
- removed joint Rigid 22
- removed joint Rigid 23
- removed joint Rigid 24
- removed joint Rigid 25
- removed joint Rigid 26
- removed joint Rigid 27
- added joint Revolute 17: type continuous, parent top_bottom_connector_5, child motor_holder_5, origin xyz=0.052 0.0325 0.0075 rpy=0 0 0, axis 1.0 0.0 0.0
- added joint Revolute 18: type continuous, parent motor_holder_5, child left_feet_connect_5, origin xyz=-0.023 0.0 -0.030252 rpy=0 0 0, axis 0.0 0.0 -1.0
- added joint Revolute 21: type continuous, parent top_bottom_connector_7, child motor_holder_7, origin xyz=-0.052 0.0325 0.0075 rpy=0 0 0, axis 1.0 0.0 0.0
- added joint Revolute 22: type continuous, parent top_bottom_connector_6, child motor_holder_6, origin xyz=0.004 0.0325 0.0075 rpy=0 0 0, axis 1.0 0.0 0.0
- added joint Revolute 23: type continuous, parent motor_holder_6, child left_feet_connect_6, origin xyz=0.023 0.0 -0.030252 rpy=0 0 0, axis 0.0 0.0 -1.0
- added joint Revolute 24: type continuous, parent motor_holder_7, child left_feet_connect_4, origin xyz=0.023 0.0 -0.03025 rpy=0 0 0, axis 0.0 0.0 -1.0
- added joint Revolute 25: type continuous, parent left_feet_connect_5, child left_feet_3, origin xyz=-0.0845 0.0 -0.0165 rpy=0 0 0, axis 0.0 0.0 -1.0
- added joint Revolute 26: type continuous, parent left_feet_connect_6, child left_feet_2, origin xyz=-0.0845 0.0 -0.0165 rpy=0 0 0, axis 0.0 0.0 -1.0
- added joint Revolute 27: type continuous, parent left_feet_connect_4, child left_feet_1, origin xyz=-0.0845 0.0 -0.0165 rpy=0 0 0, axis 0.0 0.0 -1.0

File: test_7_description/test_7_description/urdf/test_7.xacro (robot description, xacro)
@@ -578,13 +578,15 @@
   <child link="top_bottom_connector_5"/>
 </joint>
-<joint name="Rigid 17" type="fixed">
+<joint name="Revolute 17" type="continuous">
   <origin xyz="0.052 0.0325 0.0075" rpy="0 0 0"/>
   <parent link="top_bottom_connector_5"/>
   <child link="motor_holder_5"/>
-</joint>
-<joint name="Rigid 18" type="fixed">
+  <axis xyz="1.0 0.0 0.0"/>
+</joint>
+<joint name="Revolute 18" type="continuous">
   <origin xyz="-0.023 0.0 -0.030252" rpy="0 0 0"/>
   <parent link="motor_holder_5"/>
   <child link="left_feet_connect_5"/>
+  <axis xyz="0.0 0.0 -1.0"/>
 </joint>
 <joint name="Rigid 19" type="fixed">
@@ -598,38 +600,45 @@
   <child link="top_bottom_connector_7"/>
 </joint>
-<joint name="Rigid 21" type="fixed">
+<joint name="Revolute 21" type="continuous">
   <origin xyz="-0.052 0.0325 0.0075" rpy="0 0 0"/>
   <parent link="top_bottom_connector_7"/>
   <child link="motor_holder_7"/>
-</joint>
-<joint name="Rigid 22" type="fixed">
+  <axis xyz="1.0 0.0 0.0"/>
+</joint>
+<joint name="Revolute 22" type="continuous">
   <origin xyz="0.004 0.0325 0.0075" rpy="0 0 0"/>
   <parent link="top_bottom_connector_6"/>
   <child link="motor_holder_6"/>
-</joint>
-<joint name="Rigid 23" type="fixed">
+  <axis xyz="1.0 0.0 0.0"/>
+</joint>
+<joint name="Revolute 23" type="continuous">
   <origin xyz="0.023 0.0 -0.030252" rpy="0 0 0"/>
   <parent link="motor_holder_6"/>
   <child link="left_feet_connect_6"/>
-</joint>
-<joint name="Rigid 24" type="fixed">
+  <axis xyz="0.0 0.0 -1.0"/>
+</joint>
+<joint name="Revolute 24" type="continuous">
   <origin xyz="0.023 0.0 -0.03025" rpy="0 0 0"/>
   <parent link="motor_holder_7"/>
   <child link="left_feet_connect_4"/>
-</joint>
-<joint name="Rigid 25" type="fixed">
+  <axis xyz="0.0 0.0 -1.0"/>
+</joint>
+<joint name="Revolute 25" type="continuous">
   <origin xyz="-0.0845 0.0 -0.0165" rpy="0 0 0"/>
   <parent link="left_feet_connect_5"/>
   <child link="left_feet_3"/>
-</joint>
-<joint name="Rigid 26" type="fixed">
+  <axis xyz="0.0 0.0 -1.0"/>
+</joint>
+<joint name="Revolute 26" type="continuous">
   <origin xyz="-0.0845 0.0 -0.0165" rpy="0 0 0"/>
   <parent link="left_feet_connect_6"/>
   <child link="left_feet_2"/>
-</joint>
-<joint name="Rigid 27" type="fixed">
+  <axis xyz="0.0 0.0 -1.0"/>
+</joint>
+<joint name="Revolute 27" type="continuous">
   <origin xyz="-0.0845 0.0 -0.0165" rpy="0 0 0"/>
   <parent link="left_feet_connect_4"/>
   <child link="left_feet_1"/>
+  <axis xyz="0.0 0.0 -1.0"/>
 </joint>
 </robot>
